File: kicad/motion_detector/motion_detector.sch (KiCad schematic (older format))
At the start: 15 parts, among them SW1 SW_Push, U1 MPU9250, U2 AE-FT234X, U3 pic16f18326, U4 tactile_sw, U5 EEPROM, U6 character_lcd

Commit message: update
Parts:
- removed R3: 10k, symbol R
- added R?: R, symbol R
Connections:
- net +5V: now also R?.1; no longer U3.11 (RA2), U4.1
- net GND: now also 0.1pF2.1, U4.4
- new net: R?.2, U3.11 (RA2), U4.1
Changed lines of the file:
@@
-$EndComp
-$Comp
-L R R3
-U 1 1 5B539CE2
-P 6200 6650
-F 0 "R3" V 6280 6650 50  0000 C CNN
-F 1 "10k" V 6200 6650 50  0000 C CNN
-F 2 "" V 6130 6650 50  0001 C CNN
-F 3 "" H 6200 6650 50  0001 C CNN
-	1    6200 6650
-	0    1    1    0
 $EndComp
 $Comp
@@
 	4000 3800 3900 3800
 Wire Wire Line
-	4000 2500 4000 3050
-Wire Wire Line
-	4000 3050 4000 3800
+	4000 2500 4000 3800
 Wire Wire Line
 	4000 3050 4200 3050
 Wire Wire Line
-	3350 4350 3350 4550
-Wire Wire Line
-	3350 4550 3350 5200
-Wire Wire Line
-	3650 1100 3650 2050
-Wire Wire Line
-	3650 2050 3650 2750
-Wire Wire Line
-	3650 2750 4150 2750
-Wire Wire Line
-	4150 2750 4200 2750
-Wire Wire Line
-	5800 2750 5850 2750
-Wire Wire Line
-	5850 2750 6600 2750
+	3350 4350 3350 5200
+Wire Wire Line
+	3650 1100 3650 2750
+Wire Wire Line
+	3650 2750 4200 2750
+Wire Wire Line
+	5800 2750 6600 2750
 Wire Wire Line
 	2100 1550 2450 1550
@@
 Connection ~ 3350 4550
 Wire Wire Line
-	5800 3150 8700 3150
-Wire Wire Line
-	8700 3150 9500 3150
-Wire Wire Line
-	5800 3250 8800 3250
-Wire Wire Line
-	8800 3250 9400 3250
+	5800 3150 9500 3150
+Wire Wire Line
+	5800 3250 9400 3250
 Wire Wire Line
 	2100 1650 3500 1650
@@
 	7950 1950 7750 1950
 Wire Wire Line
-	7750 1950 7750 2500
-Wire Wire Line
-	7750 2500 7750 2700
+	7750 1950 7750 2700
 Wire Wire Line
 	7600 1850 7950 1850
 Wire Wire Line
-	7600 1650 7600 1750
-Wire Wire Line
-	7600 1750 7600 1850
-Wire Wire Line
-	7600 1850 7600 2000
+	7600 1650 7600 2000
 Wire Wire Line
 	7950 1750 7600 1750
@@
 	6000 3050 5800 3050
 Wire Wire Line
-	6000 1100 6000 3050
-Wire Wire Line
-	6000 3050 6000 5450
-Wire Wire Line
-	5850 6650 6050 6650
-Wire Wire Line
-	6350 6650 6550 6650
+	6000 1850 6000 5450
+Wire Wire Line
+	5850 6650 6550 6650
 Wire Wire Line
 	6000 5450 4850 5450
@@
 Wire Wire Line
 	4850 6100 4900 6100
-Connection ~ 6000 3050
 Wire Wire Line
 	4900 6300 4850 6300
@@
 Wire Wire Line
 	5400 6550 5850 6550
-Connection ~ 5850 6550
 Connection ~ 8700 3150
 Wire Wire Line
@@
 	1500 6250 1800 6250
 Wire Wire Line
-	1500 5600 1500 6000
-Wire Wire Line
-	1500 6000 1500 6250
+	1500 5600 1500 6250
 Wire Wire Line
 	1800 6350 1500 6350
 Wire Wire Line
-	1500 6350 1500 7100
-Wire Wire Line
-	1500 7100 1500 7400
+	1500 6350 1500 7400
 Wire Wire Line
 	6600 2750 6600 3750
@@
 Wire Wire Line
 	5700 6300 5850 6300
-Connection ~ 5850 6300
-Wire Wire Line
-	5850 6300 5850 6550
-Wire Wire Line
-	5850 6550 5850 6650
+Wire Wire Line
+	5850 6300 5850 6650
 Connection ~ 4000 3050
 Wire Wire Line
@@
 	4000 2050 4000 2200
 Connection ~ 3650 2050
+$Comp
+L R R?
+U 1 1 5B53B926
+P 6000 1700
+F 0 "R?" V 6080 1700 50  0000 C CNN
+F 1 "R" V 6000 1700 50  0000 C CNN
+F 2 "" V 5930 1700 50  0001 C CNN
+F 3 "" H 6000 1700 50  0001 C CNN
+	1    6000 1700
+	1    0    0    -1
+$EndComp
+Wire Wire Line
+	6000 1550 6000 1100
+Connection ~ 6000 3050
+Connection ~ 5850 6550
 $EndSCHEMATC

Commit message: update
Parts:
- removed U6: character_lcd, symbol character_lcd
- added D2, D3, D4: LED, symbol LED
- added R6, R7, R8: 1k, symbol R
- gave numbers to parts that had none: 1
Connections:
- net GND: now also R6.2, R7.2, R8.2
- net at U3.12 (RA1): now also D3.2 (A)
- net at U3.13 (RA0): now also D4.2 (A)
- net at U3.8 (RC2): now also D2.2 (A)
- new net: D2.1 (K), R6.1
- new net: D3.1 (K), R7.1
- new net: D4.1 (K), R8.1
- no-connect marks 11 -> 8
Other:
- note added: "Indicator: {0, 0, 0} to [1, 1, 1} to express 0x0 to 0xf"
- note removed: "I2C pull up inside LCD"
Changed lines of the file:
@@
 $EndComp
 $Comp
-L GND #PWR10
+L GND #PWR11
 U 1 1 5B534DDB
 P 7750 2700
-F 0 "#PWR10" H 7750 2450 50  0001 C CNN
+F 0 "#PWR11" H 7750 2450 50  0001 C CNN
 F 1 "GND" H 7750 2550 50  0000 C CNN
 F 2 "" H 7750 2700 50  0001 C CNN
@@
 	1    0    0    -1
 $EndComp
-NoConn ~ 5800 3350
-NoConn ~ 5800 2950
-NoConn ~ 5800 2850
 $Comp
 L C_Small 0.1pF2
@@
 $EndComp
 $Comp
-L GND #PWR13
-U 1 1 5B53576D
-P 9450 5300
-F 0 "#PWR13" H 9450 5050 50  0001 C CNN
-F 1 "GND" H 9450 5150 50  0000 C CNN
-F 2 "" H 9450 5300 50  0001 C CNN
-F 3 "" H 9450 5300 50  0001 C CNN
-	1    9450 5300
-	1    0    0    -1
-$EndComp
-$Comp
-L +5V #PWR11
-U 1 1 5B53573D
-P 8450 4050
-F 0 "#PWR11" H 8450 3900 50  0001 C CNN
-F 1 "+5V" H 8450 4190 50  0000 C CNN
-F 2 "" H 8450 4050 50  0001 C CNN
-F 3 "" H 8450 4050 50  0001 C CNN
-	1    8450 4050
-	1    0    0    -1
-$EndComp
-$Comp
-L character_lcd U6
-U 1 1 5B531FDA
-P 8750 5000
-F 0 "U6" H 8350 4750 60  0000 C CNN
-F 1 "character_lcd" H 8750 4900 60  0000 C CNN
-F 2 "" H 8700 5000 60  0001 C CNN
-F 3 "" H 8700 5000 60  0001 C CNN
-	1    8750 5000
-	1    0    0    -1
-$EndComp
-$Comp
 L +5V #PWR1
 U 1 1 5B53CC71
@@
 	1    0    0    -1
 $EndComp
-Text Notes 8050 5500 0    60   ~ 0
-I2C pull up inside LCD
 Text Notes 750  1150 0    60   ~ 0
 I2C pull up inside the module
@@
 Wire Wire Line
 	5400 6550 5850 6550
-Connection ~ 8700 3150
-Wire Wire Line
-	8900 4450 8900 4650
-Wire Wire Line
-	9450 4450 8900 4450
-Wire Wire Line
-	9450 5300 9450 4450
-Wire Wire Line
-	8600 4450 8600 4650
-Wire Wire Line
-	8450 4450 8600 4450
-Wire Wire Line
-	8450 4050 8450 4450
-Wire Wire Line
-	8800 3250 8800 4650
-Wire Wire Line
-	8700 4650 8700 3150
-Connection ~ 8800 3250
 Wire Wire Line
 	9150 1850 9500 1850
@@
 Connection ~ 3650 2050
 $Comp
-L R R?
+L R R3
 U 1 1 5B53B926
 P 6000 1700
-F 0 "R?" V 6080 1700 50  0000 C CNN
+F 0 "R3" V 6080 1700 50  0000 C CNN
 F 1 "R" V 6000 1700 50  0000 C CNN
 F 2 "" V 5930 1700 50  0001 C CNN
@@
 Connection ~ 6000 3050
 Connection ~ 5850 6550
+$Comp
+L LED D2
+U 1 1 5B53F757
+P 6900 4650
+F 0 "D2" H 6900 4750 50  0000 C CNN
+F 1 "LED" H 6900 4550 50  0000 C CNN
+F 2 "" H 6900 4650 50  0001 C CNN
+F 3 "" H 6900 4650 50  0001 C CNN
+	1    6900 4650
+	0    -1   -1   0
+$EndComp
+$Comp
+L LED D3
+U 1 1 5B53F790
+P 7200 4650
+F 0 "D3" H 7200 4750 50  0000 C CNN
+F 1 "LED" H 7200 4550 50  0000 C CNN
+F 2 "" H 7200 4650 50  0001 C CNN
+F 3 "" H 7200 4650 50  0001 C CNN
+	1    7200 4650
+	0    -1   -1   0
+$EndComp
+$Comp
+L LED D4
+U 1 1 5B53F7CB
+P 7500 4650
+F 0 "D4" H 7500 4750 50  0000 C CNN
+F 1 "LED" H 7500 4550 50  0000 C CNN
+F 2 "" H 7500 4650 50  0001 C CNN
+F 3 "" H 7500 4650 50  0001 C CNN
+	1    7500 4650
+	0    -1   -1   0
+$EndComp
+$Comp
+L R R6
+U 1 1 5B53F808
+P 6900 5250
+F 0 "R6" V 6980 5250 50  0000 C CNN
+F 1 "1k" V 6900 5250 50  0000 C CNN
+F 2 "" V 6830 5250 50  0001 C CNN
+F 3 "" H 6900 5250 50  0001 C CNN
+	1    6900 5250
+	1    0    0    -1
+$EndComp
+$Comp
+L R R7
+U 1 1 5B53F875
+P 7200 5250
+F 0 "R7" V 7280 5250 50  0000 C CNN
+F 1 "1k" V 7200 5250 50  0000 C CNN
+F 2 "" V 7130 5250 50  0001 C CNN
+F 3 "" H 7200 5250 50  0001 C CNN
+	1    7200 5250
+	1    0    0    -1
+$EndComp
+$Comp
+L R R8
+U 1 1 5B53F8B4
+P 7500 5250
+F 0 "R8" V 7580 5250 50  0000 C CNN
+F 1 "1k" V 7500 5250 50  0000 C CNN
+F 2 "" V 7430 5250 50  0001 C CNN
+F 3 "" H 7500 5250 50  0001 C CNN
+	1    7500 5250
+	1    0    0    -1
+$EndComp
+Wire Wire Line
+	5800 2850 7500 2850
+Wire Wire Line
+	7500 2850 7500 4500
+Wire Wire Line
+	5800 2950 7200 2950
+Wire Wire Line
+	7200 2950 7200 4500
+Wire Wire Line
+	5800 3350 6900 3350
+Wire Wire Line
+	6900 3350 6900 4500
+Wire Wire Line
+	6900 4800 6900 5100
+Wire Wire Line
+	7200 4800 7200 5100
+Wire Wire Line
+	7500 4800 7500 5100
+$Comp
+L GND #PWR10
+U 1 1 5B53FE08
+P 7200 6100
+F 0 "#PWR10" H 7200 5850 50  0001 C CNN
+F 1 "GND" H 7200 5950 50  0000 C CNN
+F 2 "" H 7200 6100 50  0001 C CNN
+F 3 "" H 7200 6100 50  0001 C CNN
+	1    7200 6100
+	1    0    0    -1
+$EndComp
+Wire Wire Line
+	6900 5400 6900 5850
+Wire Wire Line
+	6900 5850 7500 5850
+Wire Wire Line
+	7200 5400 7200 6100
+Connection ~ 7200 5850
+Wire Wire Line
+	7500 5850 7500 5400
+Text Notes 7850 4650 0    60   ~ 0
+Indicator: {0, 0, 0} to [1, 1, 1} to express 0x0 to 0xf
+Wire Notes Line
+	6650 4400 6650 4950
+Wire Notes Line
+	6650 4950 7750 4950
+Wire Notes Line
+	7750 4950 7750 4400
+Wire Notes Line
+	7750 4400 6650 4400
 $EndSCHEMATC
