File: kicad/motion_detector/motion_detector.sch (KiCad schematic (older format))
At the start: 21 parts, among them SW1 SW_Push, U1 MPU9250, U2 AE-FT234X, U3 pic16f18326, U4 tactile_sw, U5 EEPROM

Commit message: update
Parts:
- added JP1: jumper, symbol Jumper_NO_Small
- added U2: hall_sensor, symbol hall_sensor
- R8, R9: value R -> 10k
- renumbered U2 to U3, U3 to U4, U4 to U5, U5 to U6
Connections:
- net +5V: now also U2.1 (VCC)
- net GND: now also U2.3 (GND)
- net at U4.7 (RC3): now also JP1.1, U2.2 (VOUT); no longer D1.2 (A)
- new net: D1.2 (A), JP1.2
Other:
- note added: "Magnet\n"
- moved on the sheet: D1, R3
Changed lines of the file:
@@
 Sheet 1 1
 Title "Motion sensor"
-Date "2018-07-24"
-Rev "v0.2"
+Date "2018-07-25"
+Rev "v0.3"
 Comp "https://github.com/araobp"
 Comment1 ""
-Comment2 ""
+Comment2 "Allegro hall sensor"
 Comment3 "Atmel 256kbits EEPROM (I2C)"
 Comment4 "TDK InvenSense nine-axis sensor (I2C)"
 $EndDescr
 $Comp
-L pic16f18326 U3
+L pic16f18326 U4
 U 1 1 5B531F88
 P 5000 3050
-F 0 "U3" H 4450 3500 60  0000 C CNN
+F 0 "U4" H 4450 3500 60  0000 C CNN
 F 1 "pic16f18326" H 5000 3050 60  0000 C CNN
 F 2 "" H 4600 3100 60  0001 C CNN
@@
 $EndComp
 $Comp
-L AE-FT234X U2
+L AE-FT234X U3
 U 1 1 5B531FAF
 P 2500 6450
-F 0 "U2" H 2100 6800 60  0000 C CNN
+F 0 "U3" H 2100 6800 60  0000 C CNN
 F 1 "AE-FT234X" H 2550 6500 60  0000 C CNN
 F 2 "" H 2350 6450 60  0001 C CNN
@@
 $EndComp
 $Comp
-L tactile_sw U4
+L tactile_sw U5
 U 1 1 5B532037
 P 5300 6200
-F 0 "U4" H 5100 6400 60  0000 C CNN
+F 0 "U5" H 5100 6400 60  0000 C CNN
 F 1 "tactile_sw" H 5300 6200 60  0000 C CNN
 F 2 "" H 5250 6150 60  0001 C CNN
@@
 $EndComp
 $Comp
-L EEPROM U5
+L EEPROM U6
 U 1 1 5B532054
 P 8550 1800
-F 0 "U5" H 8250 2100 60  0000 C CNN
+F 0 "U6" H 8250 2100 60  0000 C CNN
 F 1 "EEPROM" H 8550 1800 60  0000 C CNN
 F 2 "" H 8450 1800 60  0001 C CNN
@@
 $EndComp
 $Comp
-L +5V #PWR6
+L +5V #PWR8
 U 1 1 5B5321A8
 P 3650 1100
-F 0 "#PWR6" H 3650 950 50  0001 C CNN
+F 0 "#PWR8" H 3650 950 50  0001 C CNN
 F 1 "+5V" H 3650 1240 50  0000 C CNN
 F 2 "" H 3650 1100 50  0001 C CNN
@@
 $EndComp
 $Comp
-L GND #PWR8
+L GND #PWR10
 U 1 1 5B532208
 P 6550 7150
-F 0 "#PWR8" H 6550 6900 50  0001 C CNN
+F 0 "#PWR10" H 6550 6900 50  0001 C CNN
 F 1 "GND" H 6550 7000 50  0000 C CNN
 F 2 "" H 6550 7150 50  0001 C CNN
@@
 $EndComp
 $Comp
-L GND #PWR5
+L GND #PWR7
 U 1 1 5B5324D1
 P 3350 5200
-F 0 "#PWR5" H 3350 4950 50  0001 C CNN
+F 0 "#PWR7" H 3350 4950 50  0001 C CNN
 F 1 "GND" H 3350 5050 50  0000 C CNN
 F 2 "" H 3350 5200 50  0001 C CNN
@@
 L LED D1
 U 1 1 5B533E19
-P 4150 3850
-F 0 "D1" H 4150 3950 50  0000 C CNN
-F 1 "LED" H 4150 3750 50  0000 C CNN
-F 2 "" H 4150 3850 50  0001 C CNN
-F 3 "" H 4150 3850 50  0001 C CNN
-	1    4150 3850
+P 4150 4000
+F 0 "D1" H 4150 4100 50  0000 C CNN
+F 1 "LED" H 4150 3900 50  0000 C CNN
+F 2 "" H 4150 4000 50  0001 C CNN
+F 3 "" H 4150 4000 50  0001 C CNN
+	1    4150 4000
 	0    -1   -1   0
 $EndComp
@@
 L R R3
 U 1 1 5B533F63
-P 4150 4250
-F 0 "R3" V 4230 4250 50  0000 C CNN
-F 1 "1k" V 4150 4250 50  0000 C CNN
-F 2 "" V 4080 4250 50  0001 C CNN
-F 3 "" H 4150 4250 50  0001 C CNN
-	1    4150 4250
+P 4150 4350
+F 0 "R3" V 4230 4350 50  0000 C CNN
+F 1 "1k" V 4150 4350 50  0000 C CNN
+F 2 "" V 4080 4350 50  0001 C CNN
+F 3 "" H 4150 4350 50  0001 C CNN
+	1    4150 4350
 	1    0    0    -1
 $EndComp
@@
 $EndComp
 $Comp
-L +5V #PWR12
+L +5V #PWR14
 U 1 1 5B534D44
 P 9300 1100
-F 0 "#PWR12" H 9300 950 50  0001 C CNN
+F 0 "#PWR14" H 9300 950 50  0001 C CNN
 F 1 "+5V" H 9300 1240 50  0000 C CNN
 F 2 "" H 9300 1100 50  0001 C CNN
@@
 $EndComp
 $Comp
-L GND #PWR11
+L GND #PWR13
 U 1 1 5B534DDB
 P 7600 2450
-F 0 "#PWR11" H 7600 2200 50  0001 C CNN
+F 0 "#PWR13" H 7600 2200 50  0001 C CNN
 F 1 "GND" H 7600 2300 50  0000 C CNN
 F 2 "" H 7600 2450 50  0001 C CNN
@@
 $EndComp
 $Comp
-L +5V #PWR7
+L +5V #PWR9
 U 1 1 5B53674E
 P 6000 1100
-F 0 "#PWR7" H 6000 950 50  0001 C CNN
+F 0 "#PWR9" H 6000 950 50  0001 C CNN
 F 1 "+5V" H 6000 1240 50  0000 C CNN
 F 2 "" H 6000 1100 50  0001 C CNN
@@
 $EndComp
 $Comp
-L GND #PWR9
+L GND #PWR11
 U 1 1 5B53CE48
 P 6600 3750
-F 0 "#PWR9" H 6600 3500 50  0001 C CNN
+F 0 "#PWR11" H 6600 3500 50  0001 C CNN
 F 1 "GND" H 6600 3600 50  0000 C CNN
 F 2 "" H 6600 3750 50  0001 C CNN
@@
 $EndComp
 $Comp
-L GND #PWR10
+L GND #PWR12
 U 1 1 5B53FE08
 P 7200 6100
-F 0 "#PWR10" H 7200 5850 50  0001 C CNN
+F 0 "#PWR12" H 7200 5850 50  0001 C CNN
 F 1 "GND" H 7200 5950 50  0000 C CNN
 F 2 "" H 7200 6100 50  0001 C CNN
@@
 	4000 3800 3900 3800
 Wire Wire Line
-	4000 2500 4000 3050
-Wire Wire Line
-	4000 3050 4000 3800
+	4000 2500 4000 3800
 Wire Wire Line
 	4000 3050 4200 3050
 Wire Wire Line
-	3350 4350 3350 4550
-Wire Wire Line
-	3350 4550 3350 5200
-Wire Wire Line
-	3650 1100 3650 2050
-Wire Wire Line
-	3650 2050 3650 2750
-Wire Wire Line
-	3650 2750 4150 2750
-Wire Wire Line
-	4150 2750 4200 2750
-Wire Wire Line
-	5800 2750 5850 2750
-Wire Wire Line
-	5850 2750 6600 2750
+	3350 4350 3350 5200
+Wire Wire Line
+	3650 1100 3650 2750
+Wire Wire Line
+	3650 2750 4200 2750
+Wire Wire Line
+	5800 2750 6600 2750
 Wire Wire Line
 	2100 1550 2450 1550
 Wire Wire Line
-	4200 3350 4150 3350
-Wire Wire Line
-	4150 3350 4150 3700
-Wire Wire Line
-	4150 4000 4150 4100
-Wire Wire Line
-	4150 4400 4150 4550
+	3000 3350 4200 3350
+Wire Wire Line
+	4150 4150 4150 4200
+Wire Wire Line
+	4150 4500 4150 4550
 Wire Wire Line
 	4150 4550 3350 4550
 Connection ~ 3350 4550
 Wire Wire Line
-	5800 3150 9500 3150
-Wire Wire Line
-	9500 3150 10100 3150
-Wire Wire Line
-	5800 3250 9400 3250
-Wire Wire Line
-	9400 3250 10350 3250
+	5800 3150 10100 3150
+Wire Wire Line
+	5800 3250 10350 3250
 Wire Wire Line
 	2100 1650 3500 1650
@@
 	7600 1850 7950 1850
 Wire Wire Line
-	7600 1650 7600 1750
-Wire Wire Line
-	7600 1750 7600 1850
-Wire Wire Line
-	7600 1850 7600 1950
-Wire Wire Line
-	7600 1950 7600 2150
-Wire Wire Line
-	7600 2150 7600 2450
+	7600 1650 7600 2450
 Wire Wire Line
 	7950 1750 7600 1750
@@
 	1500 6250 1800 6250
 Wire Wire Line
-	1500 5600 1500 6000
-Wire Wire Line
-	1500 6000 1500 6250
+	1500 5600 1500 6250
 Wire Wire Line
 	1800 6350 1500 6350
 Wire Wire Line
-	1500 6350 1500 7100
-Wire Wire Line
-	1500 7100 1500 7400
+	1500 6350 1500 7400
 Wire Wire Line
 	6600 2750 6600 3750
@@
 	5700 6300 5850 6300
 Wire Wire Line
-	5850 6300 5850 6550
-Wire Wire Line
-	5850 6550 5850 6650
+	5850 6300 5850 6650
 Connection ~ 4000 3050
 Wire Wire Line
@@
 	6900 5400 6900 5850
 Wire Wire Line
-	6900 5850 7200 5850
-Wire Wire Line
-	7200 5850 7500 5850
-Wire Wire Line
-	7200 5400 7200 5850
-Wire Wire Line
-	7200 5850 7200 6100
+	6900 5850 7500 5850
+Wire Wire Line
+	7200 5400 7200 6100
 Connection ~ 7200 5850
 Wire Wire Line
@@
 	5800 3350 6000 3350
 Wire Wire Line
-	6000 1850 6000 3350
-Wire Wire Line
-	6000 3350 6000 5250
+	6000 1850 6000 5250
 Wire Wire Line
 	6000 5250 4850 5250
@@
 P 10100 1950
 F 0 "R8" V 10180 1950 50  0000 C CNN
-F 1 "R" V 10100 1950 50  0000 C CNN
+F 1 "10k" V 10100 1950 50  0000 C CNN
 F 2 "" V 10030 1950 50  0001 C CNN
 F 3 "" H 10100 1950 50  0001 C CNN
@@
 P 10350 1950
 F 0 "R9" V 10430 1950 50  0000 C CNN
-F 1 "R" V 10350 1950 50  0000 C CNN
+F 1 "10k" V 10350 1950 50  0000 C CNN
 F 2 "" V 10280 1950 50  0001 C CNN
 F 3 "" H 10350 1950 50  0001 C CNN
@@
 Connection ~ 9400 3250
 $Comp
-L +5V #PWR13
+L +5V #PWR15
 U 1 1 5B56687B
 P 10100 1100
-F 0 "#PWR13" H 10100 950 50  0001 C CNN
+F 0 "#PWR15" H 10100 950 50  0001 C CNN
 F 1 "+5V" H 10100 1240 50  0000 C CNN
 F 2 "" H 10100 1100 50  0001 C CNN
@@
 $EndComp
 $Comp
-L +5V #PWR14
+L +5V #PWR16
 U 1 1 5B5668BB
 P 10350 1100
-F 0 "#PWR14" H 10350 950 50  0001 C CNN
+F 0 "#PWR16" H 10350 950 50  0001 C CNN
 F 1 "+5V" H 10350 1240 50  0000 C CNN
 F 2 "" H 10350 1100 50  0001 C CNN
@@
 Text Notes 4950 5800 0    60   ~ 0
 Push to start measurement for 3 sec
+$Comp
+L hall_sensor U2
+U 1 1 5B577A60
+P 2050 4150
+F 0 "U2" H 1800 4300 60  0000 C CNN
+F 1 "hall_sensor" H 2000 3900 60  0000 C CNN
+F 2 "" H 2050 4150 60  0001 C CNN
+F 3 "" H 2050 4150 60  0001 C CNN
+	1    2050 4150
+	1    0    0    -1
+$EndComp
+$Comp
+L Jumper_NO_Small JP1
+U 1 1 5B577B99
+P 4150 3750
+F 0 "JP1" H 4150 3830 50  0000 C CNN
+F 1 "jumper" H 4160 3690 50  0000 C CNN
+F 2 "" H 4150 3750 50  0001 C CNN
+F 3 "" H 4150 3750 50  0001 C CNN
+	1    4150 3750
+	0    1    1    0
+$EndComp
+Wire Wire Line
+	4150 3350 4150 3650
+Wire Wire Line
+	4150 3850 4150 3850
+Connection ~ 4150 3350
+$Comp
+L GND #PWR6
+U 1 1 5B578865
+P 2650 4750
+F 0 "#PWR6" H 2650 4500 50  0001 C CNN
+F 1 "GND" H 2650 4600 50  0000 C CNN
+F 2 "" H 2650 4750 50  0001 C CNN
+F 3 "" H 2650 4750 50  0001 C CNN
+	1    2650 4750
+	1    0    0    -1
+$EndComp
+$Comp
+L +5V #PWR5
+U 1 1 5B5788A7
+P 2650 3800
+F 0 "#PWR5" H 2650 3650 50  0001 C CNN
+F 1 "+5V" H 2650 3940 50  0000 C CNN
+F 2 "" H 2650 3800 50  0001 C CNN
+F 3 "" H 2650 3800 50  0001 C CNN
+	1    2650 3800
+	1    0    0    -1
+$EndComp
+Wire Wire Line
+	2650 3800 2650 4100
+Wire Wire Line
+	2650 4100 2550 4100
+Wire Wire Line
+	2550 4200 2650 4200
+Wire Wire Line
+	2650 4200 2650 4750
+Wire Wire Line
+	2550 4300 3000 4300
+Wire Wire Line
+	3000 4300 3000 3350
+Wire Notes Line
+	1500 4300 1500 4100
+Wire Notes Line
+	1500 4100 1650 4100
+Wire Notes Line
+	1650 4100 1650 4300
+Wire Notes Line
+	1650 4300 1500 4300
+Text Notes 1350 4400 0    60   ~ 0
+Magnet\n
 $EndSCHEMATC

Commit message: update
Parts:
- removed JP1: jumper, symbol Jumper_NO_Small
- removed U2: hall_sensor, symbol hall_sensor
- added JP1: Jumper, symbol Jumper_NC_Small
- added U6: speed_sensor, symbol speed_sensor
- renumbered U3 to U2, U4 to U3, U5 to U4, U6 to U5
Connections:
- net +5V: now also U6.1 (VDD)
- net GND: now also U6.6 (GND)
- net at R8.2, U3.10 (RC0), U5.6 (SCL): now also U6.5 (SCL)
- net at U3.7 (RC3): now also JP1.1
- net at R9.2, U3.9 (RC1), U5.5 (SDA): now also U6.4 (SDA)
- net at D1.2 (A): now also JP1.2
- no-connect marks 7 -> 9
