File: kicad/motion_detector/motion_sensor.kicad_pcb (KiCad board)
At the start: 2 copper layers, 19 parts, among them J1 Conn_01x04_Female, J2 Conn_01x02_Male, J3 Conn_01x04_Female, U1 MPU9250, U2 pic16f18326, U3 EEPROM

Commit message: update
Parts:
- moved J2 55.4 mm to (170.2, 92.7), turned to 90 degrees
- moved R6 55.1 mm to (170.2, 80.0)
- moved R5 54.0 mm to (165.1, 80.0)
- moved D4 52.9 mm to (170.2, 72.4)
- moved R4 52.9 mm to (160.0, 80.0)
- moved D3 51.7 mm to (165.1, 72.4)
- moved D2 50.6 mm to (160.0, 72.4)
- moved R8 46.9 mm to (160.0, 102.9)
- moved R7 43.2 mm to (162.6, 102.9)
- moved R2 40.7 mm to (129.5, 87.6)
- moved D1 38.1 mm to (129.5, 80.0)
- moved 0.1pF1 37.7 mm to (148.6, 61.0), turned to 180 degrees
- moved R1 36.9 mm to (142.2, 67.3)
- moved U2 36.9 mm to (148.6, 71.1)
- moved U1 35.8 mm to (144.8, 95.2)
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Routing:
- net GND: track 0.00 -> 172.7 mm, vias 0 -> 5
- net +5V: track 0.00 -> 170.2 mm, vias 0 -> 5
- net Net-(J2-Pad1): track 0.00 -> 33.0 mm, vias 0 -> 2
- net Net-(J3-Pad3): track 53.3 -> 76.2 mm, vias 0 -> 4
- net Net-(J3-Pad4): track 55.9 -> 78.7 mm, vias 0 -> 4
- net Net-(J1-Pad3): track 35.6 -> 15.2 mm, vias 2 -> 0
- net Net-(J1-Pad4): track 35.6 -> 15.2 mm, vias 2 -> 0
- net Net-(U1-Pad4): track 17.8 -> 38.1 mm, vias 0 -> 2
- net Net-(U1-Pad3): track 17.8 -> 33.0 mm, vias 0 -> 2
- net Net-(D1-Pad2): track 5.08 -> 15.2 mm
- net Net-(D2-Pad2): track 15.2 -> 7.62 mm, vias 2 -> 0
- net Net-(D3-Pad2): track 20.3 -> 15.2 mm, vias 2 -> 0
- net Net-(D4-Pad2): track 25.4 -> 22.9 mm, vias 2 -> 0
- net Net-(D1-Pad1): track 5.08 -> 2.54 mm
- net Net-(D4-Pad1): track 5.08 -> 2.54 mm
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
Commit message: update
Routing:
- net +5V: track 170.2 -> 167.6 mm, vias 5 -> 6
Changed lines of the file:
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@@
     (links 44)
     (no_connects 0)
-    (area 124.184999 58.715 185.695001 135.695)
+    (area 126.025 57.445 173.795 128.075)
     (thickness 1.6)
     (drawings 0)
-    (tracks 116)
+    (tracks 118)
     (zones 0)
     (modules 19)
@@
       (net 15 "Net-(J3-Pad4)"))
   )
+  (segment (start 132.08 71.12) (end 129.54 71.12) (width 0.25) (layer B.Cu) (net 1) (status 20))
+  (via (at 132.08 71.12) (size 0.6) (drill 0.4) (layers F.Cu B.Cu) (net 1))
+  (segment (start 132.08 81.28) (end 132.08 71.12) (width 0.25) (layer F.Cu) (net 1))
+  (segment (start 132.08 91.44) (end 132.08 81.28) (width 0.25) (layer F.Cu) (net 1))
+  (via (at 132.08 81.28) (size 0.6) (drill 0.4) (layers F.Cu B.Cu) (net 1))
+  (via (at 132.08 91.44) (size 0.6) (drill 0.4) (layers F.Cu B.Cu) (net 1))
+  (segment (start 132.08 81.28) (end 149.86 81.28) (width 0.25) (layer B.Cu) (net 1))
+  (segment (start 144.78 114.3) (end 149.86 114.3) (width 0.25) (layer B.Cu) (net 1))
   (segment (start 170.18 91.44) (end 170.18 86.36) (width 0.25) (layer B.Cu) (net 1))
   (segment (start 152.4 114.3) (end 170.18 114.3) (width 0.25) (layer B.Cu) (net 1))
-  (segment (start 149.86 81.28) (end 132.08 81.28) (width 0.25) (layer B.Cu) (net 1))
-  (via (at 132.08 81.28) (size 0.6) (drill 0.4) (layers F.Cu B.Cu) (net 1))
   (segment (start 132.08 91.44) (end 132.08 91.44) (width 0.25) (layer B.Cu) (net 1))
-  (segment (start 132.08 91.44) (end 129.54 91.44) (width 0.25) (layer B.Cu) (net 1))
+  (segment (start 132.08 91.44) (end 129.54 91.44) (width 0.25) (layer B.Cu) (net 1) (status 20))
   (segment (start 149.86 86.36) (end 149.86 114.3) (width 0.25) (layer B.Cu) (net 1))
   (segment (start 152.4 63.5) (end 149.86 63.5) (width 0.25) (layer B.Cu) (net 1))
   (segment (start 149.86 63.5) (end 149.86 81.28) (width 0.25) (layer B.Cu) (net 1))
   (segment (start 149.86 81.28) (end 149.86 86.36) (width 0.25) (layer B.Cu) (net 1))
-  (segment (start 132.08 71.12) (end 129.54 71.12) (width 0.25) (layer B.Cu) (net 1))
-  (segment (start 132.08 81.28) (end 132.08 71.12) (width 0.25) (layer F.Cu) (net 1))
-  (via (at 132.08 71.12) (size 0.6) (drill 0.4) (layers F.Cu B.Cu) (net 1))
-  (segment (start 132.08 91.44) (end 132.08 81.28) (width 0.25) (layer F.Cu) (net 1))
-  (via (at 132.08 91.44) (size 0.6) (drill 0.4) (layers F.Cu B.Cu) (net 1))
   (segment (start 160.02 83.82) (end 160.02 86.36) (width 0.25) (layer B.Cu) (net 1))
   (segment (start 165.1 83.82) (end 165.1 86.36) (width 0.25) (layer B.Cu) (net 1))
@@
   (via (at 149.86 86.36) (size 0.6) (drill 0.4) (layers F.Cu B.Cu) (net 1))
   (segment (start 149.86 86.36) (end 160.02 86.36) (width 0.25) (layer F.Cu) (net 1))
-  (segment (start 144.78 114.3) (end 149.86 114.3) (width 0.25) (layer B.Cu) (net 1))
   (segment (start 149.86 114.3) (end 152.4 114.3) (width 0.25) (layer B.Cu) (net 1))
   (segment (start 144.78 111.76) (end 144.78 114.3) (width 0.25) (layer B.Cu) (net 1))
@@
   (segment (start 152.4 60.96) (end 152.4 63.5) (width 0.25) (layer B.Cu) (net 1))
   (segment (start 144.78 86.36) (end 149.86 86.36) (width 0.25) (layer B.Cu) (net 1))
-  (segment (start 152.4 93.98) (end 152.4 109.22) (width 0.25) (layer B.Cu) (net 2))
+  (segment (start 129.54 68.58) (end 134.62 68.58) (width 0.25) (layer B.Cu) (net 2) (status 10))
+  (via (at 134.62 68.58) (size 0.6) (drill 0.4) (layers F.Cu B.Cu) (net 2))
+  (segment (start 134.62 68.58) (end 134.62 83.82) (width 0.25) (layer F.Cu) (net 2))
+  (via (at 134.62 83.82) (size 0.6) (drill 0.4) (layers F.Cu B.Cu) (net 2))
+  (segment (start 142.24 63.5) (end 129.54 63.5) (width 0.25) (layer B.Cu) (net 2))
+  (segment (start 129.54 63.5) (end 129.54 68.58) (width 0.25) (layer B.Cu) (net 2) (status 20))
+  (segment (start 152.4 96.52) (end 160.02 96.52) (width 0.25) (layer F.Cu) (net 2))
+  (via (at 160.02 96.52) (size 0.6) (drill 0.4) (layers F.Cu B.Cu) (net 2))
+  (segment (start 160.02 96.52) (end 160.02 99.06) (width 0.25) (layer B.Cu) (net 2))
+  (via (at 152.4 96.52) (size 0.6) (drill 0.4) (layers F.Cu B.Cu) (net 2))
+  (segment (start 152.4 93.98) (end 152.4 96.52) (width 0.25) (layer B.Cu) (net 2))
+  (segment (start 152.4 96.52) (end 152.4 109.22) (width 0.25) (layer B.Cu) (net 2))
   (segment (start 134.62 83.82) (end 144.78 83.82) (width 0.25) (layer B.Cu) (net 2))
   (segment (start 134.62 109.22) (end 142.24 109.22) (width 0.25) (layer B.Cu) (net 2))
+  (segment (start 134.62 83.82) (end 134.62 109.22) (width 0.25) (layer B.Cu) (net 2) (status 20))
   (via (at 152.4 109.22) (size 0.6) (drill 0.4) (layers F.Cu B.Cu) (net 2))
   (segment (start 147.32 109.22) (end 152.4 109.22) (width 0.25) (layer F.Cu) (net 2))
@@
   (segment (start 142.24 109.22) (end 147.32 109.22) (width 0.25) (layer B.Cu) (net 2))
   (segment (start 142.24 109.22) (end 142.24 109.22) (width 0.25) (layer B.Cu) (net 2))
-  (segment (start 134.62 83.82) (end 134.62 109.22) (width 0.25) (layer B.Cu) (net 2) (status 20))
   (segment (start 170.18 111.76) (end 170.18 109.22) (width 0.25) (layer B.Cu) (net 2))
   (segment (start 170.18 99.06) (end 162.56 99.06) (width 0.25) (layer B.Cu) (net 2))
@@
   (segment (start 170.18 109.22) (end 170.18 109.22) (width 0.25) (layer B.Cu) (net 2))
   (segment (start 162.56 99.06) (end 160.02 99.06) (width 0.25) (layer B.Cu) (net 2))
-  (segment (start 160.02 99.06) (end 160.02 96.52) (width 0.25) (layer B.Cu) (net 2))
-  (via (at 160.02 96.52) (size 0.6) (drill 0.4) (layers F.Cu B.Cu) (net 2))
-  (segment (start 160.02 96.52) (end 149.86 96.52) (width 0.25) (layer F.Cu) (net 2))
   (segment (start 152.4 111.76) (end 170.18 111.76) (width 0.25) (layer B.Cu) (net 2))
-  (segment (start 129.54 68.58) (end 134.62 68.58) (width 0.25) (layer B.Cu) (net 2))
-  (via (at 134.62 83.82) (size 0.6) (drill 0.4) (layers F.Cu B.Cu) (net 2))
-  (segment (start 134.62 68.58) (end 134.62 83.82) (width 0.25) (layer F.Cu) (net 2))
-  (via (at 134.62 68.58) (size 0.6) (drill 0.4) (layers F.Cu B.Cu) (net 2))
   (segment (start 152.4 111.76) (end 152.4 109.22) (width 0.25) (layer B.Cu) (net 2))
   (segment (start 147.32 60.96) (end 144.78 60.96) (width 0.25) (layer B.Cu) (net 2))
   (segment (start 144.78 60.96) (end 144.78 63.5) (width 0.25) (layer B.Cu) (net 2))
   (segment (start 144.78 63.5) (end 142.24 63.5) (width 0.25) (layer B.Cu) (net 2))
-  (segment (start 142.24 63.5) (end 129.54 63.5) (width 0.25) (layer B.Cu) (net 2))
-  (segment (start 129.54 63.5) (end 129.54 68.58) (width 0.25) (layer B.Cu) (net 2) (status 20))
-  (segment (start 129.54 81.28) (end 129.54 83.82) (width 0.25) (layer B.Cu) (net 3))
-  (segment (start 129.54 78.74) (end 144.78 78.74) (width 0.25) (layer B.Cu) (net 4))
+  (segment (start 129.54 81.28) (end 129.54 83.82) (width 0.25) (layer B.Cu) (net 3) (status 20))
+  (segment (start 129.54 78.74) (end 144.78 78.74) (width 0.25) (layer B.Cu) (net 4) (status 10))
   (segment (start 160.02 73.66) (end 160.02 76.2) (width 0.25) (layer B.Cu) (net 5))
   (segment (start 152.4 71.12) (end 160.02 71.12) (width 0.25) (layer B.Cu) (net 6))
@@
   (segment (start 152.4 66.04) (end 170.18 66.04) (width 0.25) (layer B.Cu) (net 10))
   (segment (start 170.18 66.04) (end 170.18 71.12) (width 0.25) (layer B.Cu) (net 10))
-  (segment (start 129.54 73.66) (end 144.78 73.66) (width 0.25) (layer B.Cu) (net 11))
-  (segment (start 129.54 76.2) (end 144.78 76.2) (width 0.25) (layer B.Cu) (net 12))
+  (segment (start 129.54 73.66) (end 144.78 73.66) (width 0.25) (layer B.Cu) (net 11) (status 10))
+  (segment (start 129.54 76.2) (end 144.78 76.2) (width 0.25) (layer B.Cu) (net 12) (status 10))
   (segment (start 160.02 93.98) (end 160.02 90.17) (width 0.25) (layer B.Cu) (net 13))
   (segment (start 152.4 90.17) (end 152.4 78.74) (width 0.25) (layer B.Cu) (net 13))
