File: kicad/motion_detector/motion_sensor.sch (KiCad schematic (older format))
At the start: 19 parts, among them J1 Conn_01x04_Female, J2 Conn_01x02_Male, J3 Conn_01x04_Female, U1 MPU9250, U2 pic16f18326, U3 EEPROM

Commit message: update
Other:
- note added: "Connect to USB-UART converter with 5V power supply\nor AAx3 (4.5V)"
- note removed: "Connect to USB-UART converter with 5V power supply\nor a mobile battery 5V."
Changed lines of the file:
@@
 	9950 2950 10200 2950
 Text Notes 2100 6500 0    60   ~ 0
-Connect to USB-UART converter with 5V power supply\nor a mobile battery 5V.
+Connect to USB-UART converter with 5V power supply\nor AAx3 (4.5V)
 $Comp
 L Conn_01x02_Male J2
