File: kicad/speed_sensor/speed_sensor.sch (KiCad schematic (older format))
At the start: 7 parts, among them J1 Conn_01x04_Male, U1 a1324lua-t, U2 pic16f1825

Commit message: update
Parts:
- removed U1: a1324lua-t, symbol a1324lua-t
- removed U2: pic16f1825, symbol pic16f1825
- added J2: Conn_01x03_Male, pic16f1:Pin_Header_3P, symbol Conn_01x03_Male
- added U2: pic16f18326, pic16f1:ic-pinsocket-14pins, symbol pic16f18326
- 0.1uF1: footprint (none) -> pic16f1:Capacitor
- 1k1, R1: footprint (none) -> pic16f1:Register
- D1: footprint (none) -> pic16f1:LED
- J1: footprint (none) -> pic16f1:Pin Header 4P
Connections:
- net +5V: now also J2.1 (Pin_1), U2.1 (VDD)
- net GND: now also J2.2 (Pin_2), U2.14 (VSS)
- net at J1.2 (Pin_2): now also U2.10 (RC0)
- net at R1.2: now also U2.4 (MCLR)
- net at 1k1.2: now also U2.7 (RC3)
- net at J1.1 (Pin_1): now also U2.9 (RC1)
- new net: J2.3 (Pin_3), U2.3 (RA4)
Other:
- note added: "5V"
- note added: "A1324LUA-T"
- note added: "GND\n"
- note added: "SCL"
- note added: "SDA"
Changed lines of the file:
@@
 $EndDescr
-$Comp
-L pic16f1825 U2
-U 1 1 5B5BA743
-P 5550 4050
-F 0 "U2" H 5000 4500 60  0000 C CNN
-F 1 "pic16f1825" H 5550 4050 60  0000 C CNN
-F 2 "" H 5150 4100 60  0001 C CNN
-F 3 "" H 5150 4100 60  0001 C CNN
-	1    5550 4050
-	1    0    0    -1
-$EndComp
-$Comp
-L a1324lua-t U1
-U 1 1 5B5BA862
-P 2750 3950
-F 0 "U1" H 2500 4100 60  0000 C CNN
-F 1 "a1324lua-t" H 2700 3700 60  0000 C CNN
-F 2 "" H 2750 3950 60  0001 C CNN
-F 3 "" H 2750 3950 60  0001 C CNN
-	1    2750 3950
-	1    0    0    -1
-$EndComp
 $Comp
 L +5V #PWR01
@@
 F 0 "J1" H 8200 4350 50  0000 C CNN
 F 1 "Conn_01x04_Male" H 8200 3850 50  0000 C CNN
-F 2 "" H 8200 4150 50  0001 C CNN
+F 2 "pic16f1:Pin Header 4P" H 8200 4150 50  0001 C CNN
 F 3 "" H 8200 4150 50  0001 C CNN
 	1    8200 4150
@@
 F 0 "0.1uF1" H 5560 3470 50  0000 L CNN
 F 1 "C_Small" H 5560 3320 50  0000 L CNN
-F 2 "" H 5550 3400 50  0001 C CNN
+F 2 "pic16f1:Capacitor" H 5550 3400 50  0001 C CNN
 F 3 "" H 5550 3400 50  0001 C CNN
 	1    5550 3400
@@
 F 0 "R1" V 4280 3600 50  0000 C CNN
 F 1 "51k" V 4200 3600 50  0000 C CNN
-F 2 "" V 4130 3600 50  0001 C CNN
+F 2 "pic16f1:Register" V 4130 3600 50  0001 C CNN
 F 3 "" H 4200 3600 50  0001 C CNN
 	1    4200 3600
@@
 F 0 "D1" H 3850 3100 50  0000 C CNN
 F 1 "LED" H 3850 2900 50  0000 C CNN
-F 2 "" H 3850 3000 50  0001 C CNN
+F 2 "pic16f1:LED" H 3850 3000 50  0001 C CNN
 F 3 "" H 3850 3000 50  0001 C CNN
 	1    3850 3000
@@
 F 0 "1k1" V 3930 3600 50  0000 C CNN
 F 1 "R" V 3850 3600 50  0000 C CNN
-F 2 "" V 3780 3600 50  0001 C CNN
+F 2 "pic16f1:Register" V 3780 3600 50  0001 C CNN
 F 3 "" H 3850 3600 50  0001 C CNN
 	1    3850 3600
@@
 	3850 2650 4400 2650
 Connection ~ 4400 2650
+$Comp
+L pic16f18326 U2
+U 1 1 5B77FF6D
+P 5550 4050
+F 0 "U2" H 5000 4500 60  0000 C CNN
+F 1 "pic16f18326" H 5550 4050 60  0000 C CNN
+F 2 "pic16f1:ic-pinsocket-14pins" H 5150 4100 60  0001 C CNN
+F 3 "" H 5150 4100 60  0001 C CNN
+	1    5550 4050
+	1    0    0    -1
+$EndComp
+$Comp
+L Conn_01x03_Male J2
+U 1 1 5B78015B
+P 3050 4000
+F 0 "J2" H 3050 4200 50  0000 C CNN
+F 1 "Conn_01x03_Male" H 3050 3800 50  0000 C CNN
+F 2 "pic16f1:Pin_Header_3P" H 3050 4000 50  0001 C CNN
+F 3 "" H 3050 4000 50  0001 C CNN
+	1    3050 4000
+	1    0    0    -1
+$EndComp
+Text Notes 2200 4050 0    60   ~ 0
+A1324LUA-T
+Text Notes 8250 4200 0    60   ~ 0
+SCL
+Text Notes 8250 4300 0    60   ~ 0
+SDA
+Text Notes 8250 4000 0    60   ~ 0
+5V
+Text Notes 8250 4100 0    60   ~ 0
+GND\n
 $EndSCHEMATC

Commit message: update
Other:
- note added: "4.5V-5V"
- note removed: "5V"
Changed lines of the file:
@@
 SDA
 Text Notes 8250 4000 0    60   ~ 0
-5V
+4.5V-5V
 Text Notes 8250 4100 0    60   ~ 0
 GND\n
