File: kicad/i2c_adaptor/i2c_adaptor.kicad_pcb (KiCad board)
At the start: 2 copper layers, 15 parts, among them J1 Conn_01x02, J2 Conn_01x05, J3 Conn_01x03, J4 Conn_01x14, J5 Conn_01x02, J6 Conn_01x14, Q1 Fairchild BS170, SW1 SW_SPDT, U1 pic16f1825

Commit message: update
Parts:
- added Q2: Fairchild BS170, pic16f1:BS170, F.Cu at (170.2, 102.9)
- U1: value pic16f1825 -> pic16f18326
- moved F1 12.7 mm to (186.7, 141.0)
- moved Q1 7.62 mm to (182.9, 102.9)
- moved R2 5.08 mm to (171.4, 92.7)
- moved SW1 5.08 mm to (195.6, 141.0)
- moved J2 5.08 mm to (172.7, 97.8)
- moved R3 5.08 mm to (171.4, 95.2)
Connections:
- J2 pad 2: FET -> FET2
- J3 pad 1: Net-(F1-Pad1) -> Net-(J3-Pad1)
- J4 pad 1: FET -> FET1
- J5 pad 1: Net-(J5-Pad1) -> Net-(F1-Pad2)
- Q1 pad 1: FET -> FET1
- SW1 pad 2: Net-(F1-Pad2) -> Net-(J3-Pad1)
- SW1 pad 3: Net-(J5-Pad1) -> Net-(F1-Pad1)
Routing:
- net FET: track 50.8 -> 0.00 mm, vias 2 -> 0
- net FET1: track 0.00 -> 30.5 mm
- net GND: track 91.4 -> 116.8 mm, vias 2 -> 4
- net Net-(Q2-Pad2): track 0.00 -> 20.3 mm
- net Net-(J3-Pad1): track 0.00 -> 20.3 mm
- net Net-(F1-Pad1): track 15.2 -> 5.08 mm
- net FET2: track 0.00 -> 7.62 mm
- net Net-(J5-Pad1): track 7.62 -> 0.00 mm
- net Net-(F1-Pad2): track 12.7 -> 5.08 mm
- net Net-(Q1-Pad2): track 7.62 -> 15.2 mm
- net Net-(J2-Pad5): track 22.9 -> 27.9 mm
- net Net-(J2-Pad4): track 22.9 -> 27.9 mm
- net +3V3: track 165.1 -> 160.0 mm
