File: kicad/i2c_lib_eval/i2c_lib_eval.kicad_pcb (KiCad board)
At the start: 2 copper layers, 8 parts, among them J1 Conn_01x04, J2 Conn_01x10, J3 Conn_01x06, U1 pic16f1825

Commit message: Schematic update
Connections:
- R2 pad 1: Net-(D1-Pad1) -> Net-(D1-Pad2)
- R2 pad 2: GND -> +5V
- U1 pad 7: Net-(D1-Pad2) -> Net-(D1-Pad1)
Routing:
- net GND: track 106.7 -> 101.6 mm
- net +5V: track 111.8 -> 114.4 mm, vias 4 -> 5
Changed lines of the file:
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@@
     (thickness 1.6)
     (drawings 4)
-    (tracks 54)
+    (tracks 55)
     (zones 0)
     (modules 8)
@@
     (pad_to_mask_clearance 0.05)
     (aux_axis_origin 0 0)
-    (visible_elements FFFFFF7F)
+    (visible_elements 7FFFFFFF)
     (pcbplotparams
       (layerselection 0x010fc_ffffffff)
@@
       (effects (font (size 1 1) (thickness 0.15)))
     )
+    (fp_line (start -2.54 -1.27) (end -2.54 1.27) (layer F.SilkS) (width 0.15))
+    (fp_line (start -2.54 1.27) (end 2.54 1.27) (layer F.SilkS) (width 0.15))
+    (fp_line (start 2.54 1.27) (end 2.54 -1.27) (layer F.SilkS) (width 0.15))
     (fp_line (start 2.54 -1.27) (end -2.54 -1.27) (layer F.SilkS) (width 0.15))
-    (fp_line (start 2.54 1.27) (end 2.54 -1.27) (layer F.SilkS) (width 0.15))
-    (fp_line (start -2.54 1.27) (end 2.54 1.27) (layer F.SilkS) (width 0.15))
-    (fp_line (start -2.54 -1.27) (end -2.54 1.27) (layer F.SilkS) (width 0.15))
     (pad 1 thru_hole circle (at -1.27 0 180) (size 1.524 1.524) (drill 0.762) (layers *.Cu *.Mask)
       (net 1 GND))
@@
       (effects (font (size 1 1) (thickness 0.15)))
     )
+    (fp_line (start -5.08 -1.27) (end -5.08 1.27) (layer F.SilkS) (width 0.15))
+    (fp_line (start -5.08 1.27) (end 5.08 1.27) (layer F.SilkS) (width 0.15))
+    (fp_line (start 5.08 1.27) (end 5.08 -1.27) (layer F.SilkS) (width 0.15))
     (fp_line (start 5.08 -1.27) (end -5.08 -1.27) (layer F.SilkS) (width 0.15))
-    (fp_line (start 5.08 1.27) (end 5.08 -1.27) (layer F.SilkS) (width 0.15))
-    (fp_line (start -5.08 1.27) (end 5.08 1.27) (layer F.SilkS) (width 0.15))
-    (fp_line (start -5.08 -1.27) (end -5.08 1.27) (layer F.SilkS) (width 0.15))
     (pad 1 thru_hole circle (at -3.81 0 180) (size 1.524 1.524) (drill 0.762) (layers *.Cu *.Mask)
       (net 2 +5V))
@@
       (effects (font (size 1 1) (thickness 0.15)))
     )
+    (fp_line (start -12.7 -1.27) (end -12.7 1.27) (layer F.SilkS) (width 0.15))
+    (fp_line (start -12.7 1.27) (end 12.7 1.27) (layer F.SilkS) (width 0.15))
+    (fp_line (start 12.7 1.27) (end 12.7 -1.27) (layer F.SilkS) (width 0.15))
     (fp_line (start 12.7 -1.27) (end -12.7 -1.27) (layer F.SilkS) (width 0.15))
-    (fp_line (start 12.7 1.27) (end 12.7 -1.27) (layer F.SilkS) (width 0.15))
-    (fp_line (start -12.7 1.27) (end 12.7 1.27) (layer F.SilkS) (width 0.15))
-    (fp_line (start -12.7 -1.27) (end -12.7 1.27) (layer F.SilkS) (width 0.15))
     (pad 1 thru_hole circle (at -11.43 0 270) (size 1.524 1.524) (drill 0.762) (layers *.Cu *.Mask)
       (net 2 +5V))
@@
       (effects (font (size 1 1) (thickness 0.15)))
     )
+    (fp_line (start -5.08 -1.27) (end 5.08 -1.27) (layer F.SilkS) (width 0.15))
+    (fp_line (start -5.08 -1.27) (end -5.08 1.27) (layer F.SilkS) (width 0.15))
+    (fp_line (start -5.08 1.27) (end 5.08 1.27) (layer F.SilkS) (width 0.15))
+    (fp_line (start 5.08 1.27) (end 5.08 -1.27) (layer F.SilkS) (width 0.15))
+    (pad 1 thru_hole circle (at -3.81 0 90) (size 1.524 1.524) (drill 0.762) (layers *.Cu *.Mask)
+      (net 15 "Net-(J3-Pad1)"))
+    (pad 2 thru_hole circle (at 3.81 0 90) (size 1.524 1.524) (drill 0.762) (layers *.Cu *.Mask)
+      (net 2 +5V))
+  )
+  (module pic16f1:Register (layer F.Cu)
+    (at 138.43 114.3)
+    (fp_text reference R2 (at 0 -2.54) (layer F.SilkS)
+      (effects (font (size 1 1) (thickness 0.15)))
+    )
+    (fp_text value 1k (at 0 2.54) (layer F.Fab)
+      (effects (font (size 1 1) (thickness 0.15)))
+    )
     (fp_line (start 5.08 1.27) (end 5.08 -1.27) (layer F.SilkS) (width 0.15))
     (fp_line (start -5.08 1.27) (end 5.08 1.27) (layer F.SilkS) (width 0.15))
     (fp_line (start -5.08 -1.27) (end -5.08 1.27) (layer F.SilkS) (width 0.15))
     (fp_line (start -5.08 -1.27) (end 5.08 -1.27) (layer F.SilkS) (width 0.15))
-    (pad 1 thru_hole circle (at -3.81 0 90) (size 1.524 1.524) (drill 0.762) (layers *.Cu *.Mask)
-      (net 15 "Net-(J3-Pad1)"))
-    (pad 2 thru_hole circle (at 3.81 0 90) (size 1.524 1.524) (drill 0.762) (layers *.Cu *.Mask)
-      (net 2 +5V))
-  )
-  (module pic16f1:Register (layer F.Cu)
-    (at 138.43 114.3)
-    (fp_text reference R2 (at 0 -2.54) (layer F.SilkS)
-      (effects (font (size 1 1) (thickness 0.15)))
-    )
-    (fp_text value 1k (at 0 2.54) (layer F.Fab)
-      (effects (font (size 1 1) (thickness 0.15)))
-    )
-    (fp_line (start -5.08 -1.27) (end 5.08 -1.27) (layer F.SilkS) (width 0.15))
-    (fp_line (start -5.08 -1.27) (end -5.08 1.27) (layer F.SilkS) (width 0.15))
-    (fp_line (start -5.08 1.27) (end 5.08 1.27) (layer F.SilkS) (width 0.15))
-    (fp_line (start 5.08 1.27) (end 5.08 -1.27) (layer F.SilkS) (width 0.15))
     (pad 2 thru_hole circle (at 3.81 0) (size 1.524 1.524) (drill 0.762) (layers *.Cu *.Mask)
-      (net 1 GND))
+      (net 2 +5V))
     (pad 1 thru_hole circle (at -3.81 0) (size 1.524 1.524) (drill 0.762) (layers *.Cu *.Mask)
-      (net 3 "Net-(D1-Pad1)"))
+      (net 4 "Net-(D1-Pad2)"))
   )
   (module pic16f1:ic-pinsocket-14pins (layer F.Cu)
@@
       (effects (font (size 1 1) (thickness 0.15)))
     )
+    (fp_line (start -5.08 -8.89) (end 5.08 -8.89) (layer F.SilkS) (width 0.15))
+    (fp_line (start 5.08 -8.89) (end 5.08 8.89) (layer F.SilkS) (width 0.15))
+    (fp_line (start 5.08 8.89) (end -5.08 8.89) (layer F.SilkS) (width 0.15))
     (fp_line (start -5.08 8.89) (end -5.08 -8.89) (layer F.SilkS) (width 0.15))
-    (fp_line (start 5.08 8.89) (end -5.08 8.89) (layer F.SilkS) (width 0.15))
-    (fp_line (start 5.08 -8.89) (end 5.08 8.89) (layer F.SilkS) (width 0.15))
-    (fp_line (start -5.08 -8.89) (end 5.08 -8.89) (layer F.SilkS) (width 0.15))
     (pad 1 thru_hole circle (at -3.81 -7.62) (size 1.524 1.524) (drill 0.762) (layers *.Cu *.Mask)
       (net 2 +5V))
@@
       (net 8 "Net-(J2-Pad4)"))
     (pad 7 thru_hole circle (at -3.81 7.62) (size 1.524 1.524) (drill 0.762) (layers *.Cu *.Mask)
-      (net 4 "Net-(D1-Pad2)"))
+      (net 3 "Net-(D1-Pad1)"))
     (pad 8 thru_hole circle (at 3.81 7.62) (size 1.524 1.524) (drill 0.762) (layers *.Cu *.Mask)
       (net 22 "Net-(U1-Pad8)"))
@@
       (effects (font (size 1 1) (thickness 0.15)))
     )
+    (fp_line (start -7.62 -1.27) (end -7.62 1.27) (layer F.SilkS) (width 0.15))
+    (fp_line (start -7.62 1.27) (end 7.62 1.27) (layer F.SilkS) (width 0.15))
+    (fp_line (start 7.62 1.27) (end 7.62 -1.27) (layer F.SilkS) (width 0.15))
     (fp_line (start 7.62 -1.27) (end -7.62 -1.27) (layer F.SilkS) (width 0.15))
-    (fp_line (start 7.62 1.27) (end 7.62 -1.27) (layer F.SilkS) (width 0.15))
-    (fp_line (start -7.62 1.27) (end 7.62 1.27) (layer F.SilkS) (width 0.15))
-    (fp_line (start -7.62 -1.27) (end -7.62 1.27) (layer F.SilkS) (width 0.15))
     (pad 1 thru_hole circle (at -6.35 0) (size 1.524 1.524) (drill 0.762) (layers *.Cu *.Mask)
       (net 15 "Net-(J3-Pad1)"))
@@
   (segment (start 139.7 119.38) (end 134.62 119.38) (width 0.25) (layer B.Cu) (net 1))
   (segment (start 134.62 119.38) (end 134.62 116.84) (width 0.25) (layer B.Cu) (net 1))
-  (segment (start 142.24 114.3) (end 142.24 119.38) (width 0.25) (layer B.Cu) (net 1))
   (segment (start 142.24 119.38) (end 139.7 119.38) (width 0.25) (layer B.Cu) (net 1))
   (segment (start 142.24 86.36) (end 154.94 86.36) (width 0.25) (layer B.Cu) (net 1))
@@
   (segment (start 152.4 83.82) (end 152.4 93.98) (width 0.25) (layer F.Cu) (net 2))
   (via (at 152.4 93.98) (size 0.8) (drill 0.4) (layers F.Cu B.Cu) (net 2))
+  (segment (start 142.24 114.3) (end 142.24 111.76) (width 0.25) (layer B.Cu) (net 2))
+  (via (at 142.24 111.76) (size 0.8) (drill 0.4) (layers F.Cu B.Cu) (net 2))
   (segment (start 134.62 111.76) (end 134.62 114.3) (width 0.25) (layer B.Cu) (net 3))
   (segment (start 134.62 104.14) (end 134.62 109.22) (width 0.25) (layer B.Cu) (net 4))
