File: kicad/i2c_lib_eval/i2c_lib_eval.sch (KiCad schematic (older format))
At the start: 7 parts, among them J1 Conn_01x04, J2 Conn_01x10, U1 pic16f1825

Commit message: Schemtic update
Parts:
- added J3: Conn_01x06, mcu:Pin Header 6P, symbol Connector_Generic:Conn_01x06
- C1: footprint (none) -> pic16f1:Capacitor
- D1: footprint (none) -> pic16f1:LED
- J1: footprint (none) -> mcu:pin-socket-4p
- J2: footprint (none) -> mcu:Pin Header 10P
- R1, R2: footprint (none) -> pic16f1:Register
- U1: footprint (none) -> pic16f1:ic-pinsocket-14pins
Connections:
- net +5V: now also J3.2 (Pin_2)
- net GND: now also J3.3 (Pin_3)
- net at U1.12 (RA1): now also J3.5 (Pin_5)
- net at U1.13 (RA0): now also J3.4 (Pin_4)
- net at R1.1, U1.4 (MCLR): now also J3.1 (Pin_1)
- no-connect marks 12 -> 11
Other:
- note added: "Android app with USB-OTG"
- note added: "PICkit3"
- note added: "USB Serial module (FTDI)"
- note removed: "TeraTerm on PC"
- note removed: "USB Serial module"
- moved on the sheet: D1, R1, R2
Changed lines of the file:
@@
 Sheet 1 1
 Title "Microchip I2C library evaluation board"
-Date "2020-08-11"
-Rev ""
+Date "2020-08-26"
+Rev "rev 0.3"
 Comp "https://github.com/araobp"
 Comment1 "PIC16F1825"
@@
 F 0 "U1" H 4650 5537 60  0000 C CNN
 F 1 "pic16f1825" H 4650 5431 60  0000 C CNN
-F 2 "" H 4250 5000 60  0001 C CNN
+F 2 "pic16f1:ic-pinsocket-14pins" H 4250 5000 60  0001 C CNN
 F 3 "" H 4250 5000 60  0001 C CNN
 	1    4650 4950
@@
 L Device:R R1
 U 1 1 5F325C35
-P 3450 4950
-F 0 "R1" V 3243 4950 50  0000 C CNN
-F 1 "51k" V 3334 4950 50  0000 C CNN
-F 2 "" V 3380 4950 50  0001 C CNN
-F 3 "~" H 3450 4950 50  0001 C CNN
-	1    3450 4950
+P 2700 4950
+F 0 "R1" V 2493 4950 50  0000 C CNN
+F 1 "51k" V 2584 4950 50  0000 C CNN
+F 2 "pic16f1:Register" V 2630 4950 50  0001 C CNN
+F 3 "~" H 2700 4950 50  0001 C CNN
+	1    2700 4950
 	0    1    1    0
 $EndComp
 Wire Wire Line
-	2850 4650 2850 4950
-Wire Wire Line
-	2850 4950 3300 4950
-Wire Wire Line
-	3600 4950 3850 4950
+	1700 4650 1700 4950
+Wire Wire Line
+	1700 4950 2550 4950
 $Comp
 L power:GND #PWR03
@@
 F 0 "C1" V 4421 4200 50  0000 C CNN
 F 1 "0.1uF" V 4512 4200 50  0000 C CNN
-F 2 "" H 4650 4200 50  0001 C CNN
+F 2 "pic16f1:Capacitor" H 4650 4200 50  0001 C CNN
 F 3 "~" H 4650 4200 50  0001 C CNN
 	1    4650 4200
@@
 Connection ~ 3800 4650
 Wire Wire Line
-	3800 4650 2850 4650
-Wire Wire Line
-	5500 4650 6100 4650
-Wire Wire Line
 	5450 4650 5500 4650
 Connection ~ 5500 4650
@@
 L Device:LED D1
 U 1 1 5F3277AB
-P 3450 5550
-F 0 "D1" V 3489 5432 50  0000 R CNN
-F 1 "LED" V 3398 5432 50  0000 R CNN
-F 2 "" H 3450 5550 50  0001 C CNN
-F 3 "~" H 3450 5550 50  0001 C CNN
-	1    3450 5550
+P 2550 5600
+F 0 "D1" V 2589 5482 50  0000 R CNN
+F 1 "LED" V 2498 5482 50  0000 R CNN
+F 2 "pic16f1:LED" H 2550 5600 50  0001 C CNN
+F 3 "~" H 2550 5600 50  0001 C CNN
+	1    2550 5600
 	0    -1   -1   0
 $EndComp
 Wire Wire Line
-	3850 5250 3450 5250
-Wire Wire Line
-	3450 5250 3450 5400
+	3850 5250 2550 5250
+Wire Wire Line
+	2550 5250 2550 5450
 $Comp
 L Device:R R2
 U 1 1 5F328950
-P 3450 6000
-F 0 "R2" H 3520 6046 50  0000 L CNN
-F 1 "1k" H 3520 5955 50  0000 L CNN
-F 2 "" V 3380 6000 50  0001 C CNN
-F 3 "~" H 3450 6000 50  0001 C CNN
-	1    3450 6000
-	1    0    0    -1
-$EndComp
-Wire Wire Line
-	3450 5850 3450 5700
+P 2550 6050
+F 0 "R2" H 2620 6096 50  0000 L CNN
+F 1 "1k" H 2620 6005 50  0000 L CNN
+F 2 "pic16f1:Register" V 2480 6050 50  0001 C CNN
+F 3 "~" H 2550 6050 50  0001 C CNN
+	1    2550 6050
+	1    0    0    -1
+$EndComp
+Wire Wire Line
+	2550 5900 2550 5750
 $Comp
 L power:GND #PWR02
 U 1 1 5F3290DE
-P 3450 6450
-F 0 "#PWR02" H 3450 6200 50  0001 C CNN
-F 1 "GND" H 3455 6277 50  0000 C CNN
-F 2 "" H 3450 6450 50  0001 C CNN
-F 3 "" H 3450 6450 50  0001 C CNN
-	1    3450 6450
-	1    0    0    -1
-$EndComp
-Wire Wire Line
-	3450 6150 3450 6450
+P 2550 6500
+F 0 "#PWR02" H 2550 6250 50  0001 C CNN
+F 1 "GND" H 2555 6327 50  0000 C CNN
+F 2 "" H 2550 6500 50  0001 C CNN
+F 3 "" H 2550 6500 50  0001 C CNN
+	1    2550 6500
+	1    0    0    -1
+$EndComp
+Wire Wire Line
+	2550 6200 2550 6500
 $Comp
 L Connector_Generic:Conn_01x04 J1
@@
 F 0 "J1" V 4564 1712 50  0000 R CNN
 F 1 "Conn_01x04" V 4473 1712 50  0000 R CNN
-F 2 "" H 4600 2000 50  0001 C CNN
+F 2 "mcu:pin-socket-4p" H 4600 2000 50  0001 C CNN
 F 3 "~" H 4600 2000 50  0001 C CNN
 	1    4600 2000
@@
 	5500 3650 5500 4200
 Connection ~ 5500 4200
-Text GLabel 2650 5050 0    50   Input ~ 0
+Text GLabel 1500 5050 0    50   Input ~ 0
 RX
-Text GLabel 2650 5200 0    50   Input ~ 0
+Text GLabel 1500 5200 0    50   Input ~ 0
 TX
 Text GLabel 5300 3350 2    50   Input ~ 0
@@
 	4800 3200 5300 3200
 Wire Wire Line
-	2650 5050 3850 5050
-Wire Wire Line
-	3850 5150 2900 5150
-Wire Wire Line
-	2900 5150 2900 5200
-Wire Wire Line
-	2900 5200 2650 5200
+	1500 5050 3850 5050
+Wire Wire Line
+	3850 5150 1750 5150
+Wire Wire Line
+	1750 5150 1750 5200
+Wire Wire Line
+	1750 5200 1500 5200
 NoConn ~ 3850 4750
 NoConn ~ 3850 4850
 NoConn ~ 5450 5250
 NoConn ~ 5450 4950
-NoConn ~ 5450 4850
-NoConn ~ 5450 4750
 Text Notes 4300 1900 0    50   ~ 0
-USB Serial module
-Text Notes 4350 1200 0    50   ~ 0
-TeraTerm on PC
+USB Serial module (FTDI)
+Text Notes 4100 1200 0    50   ~ 0
+Android app with USB-OTG
 Wire Notes Line
 	4650 1750 4650 1250
@@
 F 0 "J2" H 7930 4992 50  0000 L CNN
 F 1 "Conn_01x10" H 7930 4901 50  0000 L CNN
-F 2 "" H 7850 5000 50  0001 C CNN
+F 2 "mcu:Pin Header 10P" H 7850 5000 50  0001 C CNN
 F 3 "~" H 7850 5000 50  0001 C CNN
 	1    7850 5000
@@
 Wire Wire Line
 	4200 2200 4200 1700
+Wire Wire Line
+	1700 4650 3800 4650
+Wire Wire Line
+	2850 4950 3800 4950
+Wire Wire Line
+	5500 4650 6100 4650
+$Comp
+L Connector_Generic:Conn_01x06 J3
+U 1 1 5F4A345B
+P 4600 6750
+F 0 "J3" V 4472 6362 50  0000 R CNN
+F 1 "Conn_01x06" V 4563 6362 50  0000 R CNN
+F 2 "mcu:Pin Header 6P" H 4600 6750 50  0001 C CNN
+F 3 "~" H 4600 6750 50  0001 C CNN
+	1    4600 6750
+	0    -1   1    0
+$EndComp
+Wire Wire Line
+	3800 4950 3800 6300
+Wire Wire Line
+	3800 6300 4400 6300
+Wire Wire Line
+	4400 6300 4400 6550
+Connection ~ 3800 4950
+Wire Wire Line
+	3800 4950 3850 4950
+Wire Wire Line
+	4800 6400 4800 6550
+Wire Wire Line
+	5600 6400 4800 6400
+Wire Wire Line
+	4700 6300 4700 6550
+Wire Wire Line
+	5700 6300 4700 6300
+Wire Wire Line
+	5700 4750 5700 6300
+Wire Wire Line
+	5450 4850 5600 4850
+Wire Wire Line
+	5450 4750 5700 4750
+Wire Wire Line
+	5600 6400 5600 4850
+NoConn ~ 4900 6550
+Text Notes 4500 6950 0    50   ~ 0
+PICkit3
+$Comp
+L power:+5V #PWR04
+U 1 1 5F4B0DDF
+P 4500 6100
+F 0 "#PWR04" H 4500 5950 50  0001 C CNN
+F 1 "+5V" H 4515 6273 50  0000 C CNN
+F 2 "" H 4500 6100 50  0001 C CNN
+F 3 "" H 4500 6100 50  0001 C CNN
+	1    4500 6100
+	1    0    0    -1
+$EndComp
+Wire Wire Line
+	4500 6550 4500 6100
+$Comp
+L power:GND #PWR01
+U 1 1 5F4B2158
+P 4050 6950
+F 0 "#PWR01" H 4050 6700 50  0001 C CNN
+F 1 "GND" H 4055 6777 50  0000 C CNN
+F 2 "" H 4050 6950 50  0001 C CNN
+F 3 "" H 4050 6950 50  0001 C CNN
+	1    4050 6950
+	1    0    0    -1
+$EndComp
+Wire Wire Line
+	4600 6550 4600 6450
+Wire Wire Line
+	4600 6450 4050 6450
+Wire Wire Line
+	4050 6450 4050 6950
 $EndSCHEMATC

Commit message: Schematic update
Connections:
- net +5V: now also R2.2
- net GND: no longer R2.2
- net at U1.7 (RC3): now also D1.1 (K); no longer D1.2 (A)
- net at R2.1: now also D1.2 (A); no longer D1.1 (K)
Other:
- note added: "Status indicator"
- moved on the sheet: D1
Changed lines of the file:
@@
 Sheet 1 1
 Title "Microchip I2C library evaluation board"
-Date "2020-08-26"
-Rev "rev 0.3"
+Date "2020-08-29"
+Rev "rev 0.4"
 Comp "https://github.com/araobp"
 Comment1 "PIC16F1825"
@@
 F 3 "~" H 2550 5600 50  0001 C CNN
 	1    2550 5600
-	0    -1   -1   0
+	0    1    1    0
 $EndComp
 Wire Wire Line
@@
 Wire Wire Line
 	2550 5900 2550 5750
-$Comp
-L power:GND #PWR02
-U 1 1 5F3290DE
-P 2550 6500
-F 0 "#PWR02" H 2550 6250 50  0001 C CNN
-F 1 "GND" H 2555 6327 50  0000 C CNN
-F 2 "" H 2550 6500 50  0001 C CNN
-F 3 "" H 2550 6500 50  0001 C CNN
-	1    2550 6500
-	1    0    0    -1
-$EndComp
 Wire Wire Line
 	2550 6200 2550 6500
@@
 Wire Wire Line
 	4050 6450 4050 6950
+$Comp
+L power:+5V #PWR0103
+U 1 1 5F49DB75
+P 1950 5700
+F 0 "#PWR0103" H 1950 5550 50  0001 C CNN
+F 1 "+5V" H 1965 5873 50  0000 C CNN
+F 2 "" H 1950 5700 50  0001 C CNN
+F 3 "" H 1950 5700 50  0001 C CNN
+	1    1950 5700
+	1    0    0    -1
+$EndComp
+Wire Wire Line
+	2550 6500 1950 6500
+Wire Wire Line
+	1950 6500 1950 5700
+Text Notes 2650 5650 0    50   ~ 0
+Status indicator
 $EndSCHEMATC
